File: PCB/Athena_Mk1/Athena_Mk1.sch (KiCad schematic (older format))
At the start: 8 parts, among them J1 Power Supply, Q1 BF244B, U1 Teensy3.6, U2 RFM96W, U3 Venus634_GPS

Commit message: Replace Athena_Mk1.sch
Parts:
- added U4: 7805, TO_SOT_Packages_THT:SIPAK_Vertical, symbol 7805
- U1: footprint (none) -> RFM96W:Teensy_3.6
- U2: footprint TO_SOT_Packages_THT:TO-5-6 -> RFM96W:RFM96W
Connections:
- net labels added: +3.3V, +5V
- net labels removed: 3.3V, 5V, VIN
- wire segments 11 -> 25
- no-connect marks 83 -> 86
Other:
- moved on the sheet: BZ1, C1, D1, J1, Q1, U1, U2, U3
